File: PCB/Servomotor3/V11RC3/V11RC3.kicad_pcb (KiCad board)
At the start: 2 copper layers, 37.8 x 44.4 mm, 69 parts, among them J1 01x04 male P=1.27mm, J2 01x05 male P=1.27mm, J3 Conn_01x01_Socket, J4 Conn_01x06_Socket, J6 Conn_01x01_Socket, J7 Conn_01x01_Socket, J8 Conn_01x01_Socket, SW1 TS3735PA-250gf, SW2 TS3735PA-250gf, U1 ATD5833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

Commit message: iStrangely, this firmware does not work. Motor cannot enable and spin. DON'T USE THIS FIRMWARE. Adding a test program for testing the PID controller Adding a "Set Max allowable position deviation" command Cleaning up usage of pyserial module in upgrade_firmware.py Some refactorying of some #defines Adding a test program for "Get comprehensive position" Code improvements and bug fixes.
Parts:
- added ?: , , F.Cu at (193.8, 95.9)
- added ?: , , F.Cu at (206.9, 97.7)
- added ?: , , F.Cu at (209.9, 94.9)
- added ?: , , F.Cu at (192.0, 92.5)
